Commit message: fix error with firction

File: mobile_robot_description/urdf/macros.xacro (robot description, xacro)
@@ -39,4 +39,10 @@
         <gazebo reference="${lr}_wheel">
           <material>Gazebo/Black</material>
+            <mu1>1.0</mu1>
+            <mu2>1.0</mu2>
+            <kp>1000000.0</kp>
+            <kd>100.0</kd>
+            <minDepth>0.001</minDepth>
+            <maxVel>1.0</maxVel>
         </gazebo>
        <joint name="${lr}_wheel_hinge" type="continuous">

File: mobile_robot_description/urdf/mobile_robot.xacro (robot description, xacro)
@@ -51,12 +51,4 @@
 	<sphere radius="${casterRadius}"/>
       </geometry>
-      <surface>
-        <friction>
-          <ode>
-            <mu>0.001</mu>
-            <mu2>0.001</mu2>
-          </ode>
-        </friction>
-      </surface>
     </collision>
     <visual>
@@ -75,11 +67,4 @@
   <wheel lr="right" tY="1"/>
   	<link name="SonarFront_frame">
-              <visual>
-                <origin xyz="0 0 0" rpy="0 0 0"/>
-                    <geometry>
-                        <box size="0.01 0.01 0.05"/>
-                    </geometry>
-                    <material name="blue"/>
-                </visual>
         </link>
 	<joint name="Sonar/Front_sensor_fixedjoint" type="fixed">
@@ -89,11 +74,4 @@
 	</joint>
   	<link name="SonarLeft_frame">
-              <visual>
-                <origin xyz="0 0 0" rpy="0 0 0"/>
-                    <geometry>
-                        <box size="0.01 0.01 0.05"/>
-                    </geometry>
-                    <material name="blue"/>
-                </visual>
         </link>
 	<joint name="Sonar/Left_sensor_fixedjoint" type="fixed">
@@ -103,11 +81,4 @@
 	</joint>
   	<link name="SonarRight_frame">
-              <visual>
-                <origin xyz="0 0 0" rpy="0 0 0"/>
-                    <geometry>
-                        <box size="0.01 0.01 0.05"/>
-                    </geometry>
-                    <material name="blue"/>
-                </visual>
         </link>
 	<joint name="Sonar/Right_sensor_fixedjoint" type="fixed">
@@ -122,21 +93,4 @@
     </joint>
     <link name="imu_link">
-        <inertial>
-            <mass value="0.001"/>
-            <origin rpy="0 0 0" xyz="0 0 0"/>
-            <inertia ixx="0.0001" ixy="0" ixz="0" iyy="0.000001" iyz="0" izz="0.0001"/>
-        </inertial>
-        <visual>
-            <origin rpy="0 0 0" xyz="0 0 0"/>
-            <geometry>
-                <box size="0.001 0.001 0.001"/>
-            </geometry>
-        </visual>
-        <collision>
-            <origin rpy="0 0 0" xyz="0 0 0"/>
-            <geometry>
-                <box size=".001 .001 .001"/>
-            </geometry>
-        </collision>
     </link>
     <xacro:include filename="$(find mobile_robot_description)/urdf/mobile_robot.gazebo" />
