Commit message: add imu

File: mobile_robot_description/urdf/mobile_robot.xacro (robot description, xacro)
@@ -116,4 +116,28 @@
 		<origin rpy="0 0.0 -1.57" xyz="-0.05 -0.1 0.1"/>
 	</joint>
+    <joint name="imu_joint" type="fixed">
+        <origin xyz="0 0 0"/>
+        <parent link="chassis"/>
+        <child link="imu_link"/>
+    </joint>
+    <link name="imu_link">
+        <inertial>
+            <mass value="0.001"/>
+            <origin rpy="0 0 0" xyz="0 0 0"/>
+            <inertia ixx="0.0001" ixy="0" ixz="0" iyy="0.000001" iyz="0" izz="0.0001"/>
+        </inertial>
+        <visual>
+            <origin rpy="0 0 0" xyz="0 0 0"/>
+            <geometry>
+                <box size="0.001 0.001 0.001"/>
+            </geometry>
+        </visual>
+        <collision>
+            <origin rpy="0 0 0" xyz="0 0 0"/>
+            <geometry>
+                <box size=".001 .001 .001"/>
+            </geometry>
+        </collision>
+    </link>
     <xacro:include filename="$(find mobile_robot_description)/urdf/mobile_robot.gazebo" />
 </robot>

Commit message: modif du robot

File: mobile_robot_description/urdf/mobile_robot.xacro (robot description, xacro)
@@ -73,17 +73,31 @@
 		<origin rpy="0 0.0 0" xyz="0.2 0 0.1"/>
 	</joint>
-  	<link name="SonarLeft_frame">
+  	<link name="SonarLeftFront_frame">
         </link>
-	<joint name="Sonar/Left_sensor_fixedjoint" type="fixed">
+	<joint name="Sonar/LeftFront_sensor_fixedjoint" type="fixed">
 		<parent link="chassis"/>
-		<child link="SonarLeft_frame"/>
-		<origin rpy="0 0.0 1.57" xyz="-0.05 0.1 0.1"/>
+		<child link="SonarLeftFront_frame"/>
+		<origin rpy="0 0.0 1.57" xyz="-0.0 0.1 0.1"/>
 	</joint>
-  	<link name="SonarRight_frame">
+  	<link name="SonarLeftBack_frame">
         </link>
-	<joint name="Sonar/Right_sensor_fixedjoint" type="fixed">
+	<joint name="Sonar/LeftBack_sensor_fixedjoint" type="fixed">
 		<parent link="chassis"/>
-		<child link="SonarRight_frame"/>
-		<origin rpy="0 0.0 -1.57" xyz="-0.05 -0.1 0.1"/>
+		<child link="SonarLeftBack_frame"/>
+		<origin rpy="0 0.0 1.57" xyz="-0.2 0.1 0.1"/>
+	</joint>
+  	<link name="SonarRightFront_frame">
+        </link>
+	<joint name="Sonar/RightFront_sensor_fixedjoint" type="fixed">
+		<parent link="chassis"/>
+		<child link="SonarRightFront_frame"/>
+		<origin rpy="0 0.0 -1.57" xyz="-0.0 -0.1 0.1"/>
+	</joint>
+  	<link name="SonarRightBack_frame">
+        </link>
+	<joint name="Sonar/RightBack_sensor_fixedjoint" type="fixed">
+		<parent link="chassis"/>
+		<child link="SonarRightBack_frame"/>
+		<origin rpy="0 0.0 -1.57" xyz="-0.2 -0.1 0.1"/>
 	</joint>
     <joint name="imu_joint" type="fixed">

Commit message: evite que le capteur soit sur la roue du robot

File: mobile_robot_description/urdf/mobile_robot.xacro (robot description, xacro)
@@ -78,5 +78,5 @@
 		<parent link="chassis"/>
 		<child link="SonarLeftFront_frame"/>
-		<origin rpy="0 0.0 1.57" xyz="-0.0 0.1 0.1"/>
+		<origin rpy="0 0.0 1.57" xyz="-0.02 0.1 0.1"/>
 	</joint>
   	<link name="SonarLeftBack_frame">
@@ -92,5 +92,5 @@
 		<parent link="chassis"/>
 		<child link="SonarRightFront_frame"/>
-		<origin rpy="0 0.0 -1.57" xyz="-0.0 -0.1 0.1"/>
+		<origin rpy="0 0.0 -1.57" xyz="-0.02 -0.1 0.1"/>
 	</joint>
   	<link name="SonarRightBack_frame">
